File: kb_right.kicad_pcb (KiCad board)
At the start: 2 copper layers, 208.8 x 117.5 mm, 178 parts, among them J1 10029449-001RLF, J2 Conn_01x03, J3 Conn_01x06, J4 Conn_01x08, J5 Conn_01x09, SW0 RotaryEncoder_Switch

Commit message: start thru hole
Parts:
- moved J5 130.3 mm to (316.1, 112.0)
- moved J4 107.0 mm to (125.4, -51.4)
- moved J3 96.2 mm to (189.7, -27.0)
- moved J2 70.5 mm to (213.5, -23.4)
- moved J1 3.63 mm to (193.7, 39.3), turned to 0 degrees
- turned SW0 to -90 degrees
Routing:
- net +5V: track 1061.2 -> 0.00 mm, vias 6 -> 0
- net /ROW9: track 295.5 -> 0.00 mm, vias 2 -> 0
- net /ROW8: track 289.4 -> 0.00 mm, vias 4 -> 0
- net /ROW7: track 281.5 -> 0.00 mm, vias 4 -> 0
- net /ROW6: track 252.3 -> 0.00 mm, vias 2 -> 0
- net /ROW5: track 251.1 -> 0.00 mm, vias 2 -> 0
- net /COL0: track 248.2 -> 0.00 mm
- net /COL2: track 222.5 -> 0.00 mm, vias 6 -> 0
- net /COL1: track 218.7 -> 0.00 mm, vias 5 -> 0
- net Net-(D108-Pad2): track 215.2 -> 0.00 mm
- net /COL3: track 207.6 -> 0.00 mm, vias 6 -> 0
- net Net-(D118-Pad2): track 204.2 -> 0.00 mm
- net /COL5: track 197.8 -> 0.00 mm, vias 6 -> 0
- net Net-(D127-Pad2): track 196.5 -> 0.00 mm
- net /COL4: track 190.4 -> 0.00 mm, vias 6 -> 0
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Other:
- board size 208.8 x 117.5 mm -> 206.4 x 115.1 mm

Commit message: try again - add rgb routing
Parts:
- removed D0: D_Small, Diode_SMD:D_SOD-123
- removed SW0: RotaryEncoder_Switch, Keebio-Parts:RotaryEncoder_EC11
- added D45: D_Small, Diode_SMD:D_SOD-123, F.Cu at (167.8, -42.3)
- added D9: D_Small, Diode_SMD:D_SOD-123, F.Cu at (186.9, -47.9)
- added MX7_1: MX-NoLED, MX_Only:MXOnly-2U-Hotswap, F.Cu at (179.4, 57.1)
- added MX9: MX-NoLED, MX_Only:MXOnly-1U-Hotswap, F.Cu at (212.7, 52.4)
- added SW1: RotaryEncoder_Switch, Keebio-Parts:RotaryEncoder_EC11, F.Cu at (236.5, 52.4)
- MX7: footprint MX_Only:MXOnly-2U-Hotswap -> MX_Only:MXOnly-1U-Hotswap
- moved D10 175.3 mm to (38.1, 256.4)
- moved D11 175.3 mm to (57.1, 256.4)
- moved D12 175.3 mm to (76.2, 256.4)
- moved D13 175.3 mm to (95.2, 256.4)
- moved D14 175.3 mm to (114.3, 256.4)
- moved D15 175.3 mm to (133.3, 256.4)
- moved D16 175.3 mm to (152.4, 256.4)
- moved D17 175.3 mm to (176.2, 256.4)
- moved D18 175.3 mm to (204.8, 256.4)
- moved D27 175.3 mm to (223.8, 256.4)
- moved D28 175.3 mm to (52.4, 294.5)
- moved D29 175.3 mm to (71.4, 294.5)
- moved D30 175.3 mm to (90.5, 294.5)
- moved D31 175.3 mm to (109.5, 294.5)
- moved D32 175.3 mm to (128.6, 294.5)
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- renumbered D9 to D10, D10 to D11, D11 to D12, D12 to D13, D13 to D14, D14 to D15, D15 to D16, D16 to D17, D17 to D18, D18 to D19, D19 to D20, D20 to D21, D21 to D22, D22 to D23, D23 to D24, D24 to D25, D25 to D26, D26 to D27, D27 to D28, D28 to D29, D29 to D30, D30 to D31, D31 to D32, D32 to D35, D35 to D36, D36 to D37, D37 to D38, D38 to D39, D39 to D40, D40 to D41, D41 to D42, D42 to D43, MX9 to MX10, MX10 to MX11, MX11 to MX12, MX12 to MX13, MX13 to MX14, MX14 to MX15, MX15 to MX16, MX16 to MX17, MX17 to MX18, MX18 to MX19, MX19 to MX20, MX20 to MX21, MX21 to MX22, MX22 to MX23, MX23 to MX24, MX24 to MX25, MX25 to MX26, MX26 to MX27, MX27 to MX28, MX28 to MX29, MX29 to MX30, MX30 to MX31, MX31 to MX32, MX32_2 to MX32_1, MX32_1 to MX32_2, MX32 to MX33, MX33 to MX34, MX34 to MX35, MX35 to MX36, MX36 to MX37, MX37 to MX38, MX38 to MX39, MX39 to MX40, MX40 to MX41, MX41 to MX42, MX42 to MX43
Connections:
- D101 pad 4: /RGB_IN -> Net-(D101-Pad4)
- D102 pad 2: Net-(D102-Pad2) -> Net-(D101-Pad4)
- D102 pad 4: Net-(D101-Pad2) -> Net-(D102-Pad4)
- D103 pad 2: Net-(D103-Pad2) -> Net-(D102-Pad4)
- D103 pad 4: Net-(D102-Pad2) -> Net-(D103-Pad4)
- D104 pad 2: Net-(D104-Pad2) -> Net-(D103-Pad4)
- D104 pad 4: Net-(D103-Pad2) -> Net-(D105-Pad2)
- D105 pad 4: Net-(D104-Pad2) -> Net-(D105-Pad4)
- D106 pad 2: Net-(D106-Pad2) -> Net-(D105-Pad4)
- D106 pad 4: Net-(D105-Pad2) -> Net-(D107-Pad2)
- D107 pad 4: Net-(D106-Pad2) -> Net-(D107-Pad4)
- D108 pad 2: Net-(D108-Pad2) -> Net-(D107-Pad4)
- D108 pad 4: Net-(D107-Pad2) -> /RGB_IN
- D109 pad 4: Net-(D108-Pad2) -> Net-(D101-Pad2)
- D118 pad 2: Net-(D118-Pad2) -> Net-(D127-Pad4)
- D119 pad 4: Net-(D118-Pad2) -> Net-(D119-Pad4)
- D120 pad 2: Net-(D120-Pad2) -> Net-(D119-Pad4)
- D120 pad 4: Net-(D119-Pad2) -> Net-(D120-Pad4)
- D121 pad 2: Net-(D121-Pad2) -> Net-(D120-Pad4)
- D121 pad 4: Net-(D120-Pad2) -> Net-(D121-Pad4)
- D122 pad 2: Net-(D122-Pad2) -> Net-(D121-Pad4)
- D122 pad 4: Net-(D121-Pad2) -> Net-(D122-Pad4)
- D123 pad 2: Net-(D123-Pad2) -> Net-(D122-Pad4)
- D123 pad 4: Net-(D122-Pad2) -> Net-(D123-Pad4)
- D124 pad 2: Net-(D124-Pad2) -> Net-(D123-Pad4)
- D124 pad 4: Net-(D123-Pad2) -> Net-(D124-Pad4)
- D125 pad 2: Net-(D125-Pad2) -> Net-(D124-Pad4)
- D125 pad 4: Net-(D124-Pad2) -> Net-(D125-Pad4)
- D126 pad 2: Net-(D126-Pad2) -> Net-(D125-Pad4)
- D126 pad 4: Net-(D125-Pad2) -> Net-(D126-Pad4)
- D127 pad 2: Net-(D127-Pad2) -> Net-(D126-Pad4)
- D127 pad 4: Net-(D126-Pad2) -> Net-(D127-Pad4)
- D128 pad 4: Net-(D127-Pad2) -> Net-(D119-Pad2)
- D135 pad 2: Net-(D135-Pad2) -> unconnected-(D135-Pad2)
- D135 pad 4: Net-(D134-Pad2) -> Net-(D135-Pad4)
- D136 pad 2: Net-(D136-Pad2) -> Net-(D135-Pad4)
- D136 pad 4: Net-(D135-Pad2) -> Net-(D136-Pad4)
- D137 pad 2: Net-(D137-Pad2) -> Net-(D136-Pad4)
- D137 pad 4: Net-(D136-Pad2) -> Net-(D137-Pad4)
- D138 pad 2: Net-(D138-Pad2) -> Net-(D137-Pad4)
- D138 pad 4: Net-(D137-Pad2) -> Net-(D139-Pad2)
- D139 pad 4: Net-(D138-Pad2) -> Net-(D139-Pad4)
- D140 pad 2: Net-(D140-Pad2) -> Net-(D139-Pad4)
- D140 pad 4: Net-(D139-Pad2) -> Net-(D140-Pad4)
- D141 pad 2: Net-(D141-Pad2) -> Net-(D140-Pad4)
- D141 pad 4: Net-(D140-Pad2) -> Net-(D141-Pad4)
- D142 pad 2: unconnected-(D142-Pad2) -> Net-(D141-Pad4)
- D142 pad 4: Net-(D141-Pad2) -> Net-(D134-Pad2)
- J1 pad 1: /ROW9 -> /COL8
- J1 pad 10: /COL4 -> /ROW5
- J1 pad 11: /COL5 -> /ROW6
- J1 pad 12: /COL6 -> /ROW7
- J1 pad 13: /COL7 -> /ROW8
- J1 pad 14: /COL8 -> /ROW9
- J1 pad 2: /ROW8 -> /COL7
- J1 pad 3: /ROW7 -> /COL6
- J1 pad 4: /ROW6 -> /COL5
- J1 pad 5: /ROW5 -> /COL4
- J1 pad 6: /COL0 -> /COL3
- J1 pad 7: /COL1 -> /COL2
- J1 pad 8: /COL2 -> /COL1
- J1 pad 9: /COL3 -> /COL0
- MX37 pad 1: /COL2 -> /COL1
- MX38 pad 1: /COL3 -> /COL2
- MX39 pad 1: /COL4 -> /COL3
- MX40 pad 1: /COL5 -> /COL4
- MX41 pad 1: /COL6 -> /COL5
- MX42 pad 1: /COL7 -> /COL6
- MX43 pad 1: /COL8 -> /COL7
Routing:
- net +5V: track 0.00 -> 77.7 mm
- net Net-(D133-Pad2): track 0.00 -> 42.1 mm
- net Net-(D132-Pad2): track 0.00 -> 37.6 mm
- net Net-(D107-Pad4): track 0.00 -> 33.3 mm
- net Net-(D107-Pad2): track 0.00 -> 31.5 mm
- net Net-(D125-Pad4): track 0.00 -> 30.9 mm
- net Net-(D134-Pad2): track 0.00 -> 30.1 mm
- net Net-(D124-Pad4): track 0.00 -> 26.2 mm
- net Net-(D119-Pad2): track 0.00 -> 25.5 mm
- net Net-(D127-Pad4): track 0.00 -> 25.4 mm
- net Net-(D101-Pad2): track 0.00 -> 23.8 mm
- net Net-(D116-Pad2): track 0.00 -> 23.8 mm
- net Net-(D135-Pad4): track 0.00 -> 21.4 mm
- net Net-(D139-Pad2): track 0.00 -> 19.0 mm
- net Net-(D137-Pad4): track 0.00 -> 19.0 mm
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
Commit message: most routing done
Parts:
- D1, D10, D11, D12, D13, D14, D15, D19, D2, D20, D21, D22, D23, D24, D28, D29, D3, D30, D31, D32, D36, D37, D38, D39, D4, D40, D41, D5, D6: footprint Diode_SMD:D_SOD-123 -> Keebio-Parts:Diode-Hybrid-Back; moved to F.Cu
- D33: renamed from D35; footprint Diode_SMD:D_SOD-123 -> Keebio-Parts:Diode-Hybrid-Back; moved to F.Cu
- D44: renamed from D45; moved to B.Cu
- D9: moved to B.Cu
- moved D41 280.9 mm to (144.5, 40.5)
- moved D40 274.6 mm to (125.4, 40.5)
- moved D39 274.2 mm to (106.4, 40.5)
- moved D38 273.8 mm to (87.3, 40.5)
- moved D37 273.5 mm to (68.3, 40.5)
- moved D36 273.2 mm to (49.2, 40.5)
- moved D33 259.9 mm to (147.6, 39.7)
- moved D28 254.8 mm to (52.4, 39.7)
- moved D29 254.8 mm to (71.4, 39.7)
- moved D30 254.8 mm to (90.5, 39.7)
- moved D31 254.8 mm to (109.5, 39.7)
- moved D32 254.8 mm to (128.6, 39.7)
- moved D19 236.9 mm to (55.6, 38.9)
- moved D20 236.9 mm to (74.6, 38.9)
- moved D21 236.9 mm to (93.7, 38.9)
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- renumbered D32_1 to D33_1, D33 to D34, D34 to D35
Connections:
- J1 pad 1: /COL8 -> /COL0
- J1 pad 10: /ROW5 -> /ENC_R2
- J1 pad 11: /ROW6 -> /ENC_R1
- J1 pad 12: /ROW7 -> /ROW5
- J1 pad 13: /ROW8 -> /ROW6
- J1 pad 14: /ROW9 -> /ROW7
- J1 pad 15: /ENC_R2 -> /ROW8
- J1 pad 16: /ENC_R1 -> /ROW9
- J1 pad 2: /COL7 -> /COL1
- J1 pad 3: /COL6 -> /COL2
- J1 pad 4: /COL5 -> /COL3
- J1 pad 6: /COL3 -> /COL5
- J1 pad 7: /COL2 -> /COL6
- J1 pad 8: /COL1 -> /COL7
- J1 pad 9: /COL0 -> /COL8
Routing:
- net +5V: track 77.7 -> 989.2 mm, vias 0 -> 6
- net /COL0: track 0.00 -> 256.3 mm
- net /COL1: track 0.00 -> 247.7 mm, vias 0 -> 5
- net /COL2: track 0.00 -> 232.8 mm, vias 0 -> 5
- net /ROW9: track 0.00 -> 232.0 mm, vias 0 -> 2
- net /COL3: track 0.00 -> 217.5 mm, vias 0 -> 5
- net /COL5: track 0.00 -> 209.7 mm, vias 0 -> 5
- net /COL4: track 0.00 -> 201.0 mm, vias 0 -> 5
- net /ROW8: track 0.00 -> 196.9 mm, vias 0 -> 2
- net /COL6: track 0.00 -> 183.1 mm, vias 0 -> 6
- net /ROW7: track 0.00 -> 151.0 mm, vias 0 -> 2
- net /ROW6: track 0.00 -> 144.4 mm, vias 0 -> 2
- net Net-(D41-Pad2): track 0.00 -> 135.4 mm, vias 0 -> 1
- net /COL7: track 0.00 -> 129.2 mm, vias 0 -> 5
- net Net-(D40-Pad2): track 0.00 -> 116.7 mm, vias 0 -> 1
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Other:
- outline, holes or cut-outs redrawn
